File: MTP_PCB/MTP_PCB.kicad_pcb (KiCad board)
At the start: 2 copper layers, 65 x 56 mm, 5 parts, among them J1 GPIO

Commit message: first version PCB finished
Parts:
- added D2: LED, LED_SMD:LED_1206_3216Metric_Pad1.42x1.75mm_HandSolder, F.Cu at (130.1, 96.0)
- added D3: LED, LED_SMD:LED_1206_3216Metric_Pad1.42x1.75mm_HandSolder, F.Cu at (126.9, 96.0)
- added D4: LED, LED_SMD:LED_1206_3216Metric_Pad1.42x1.75mm_HandSolder, F.Cu at (123.3, 96.0)
- added D5: LED, LED_SMD:LED_1206_3216Metric_Pad1.42x1.75mm_HandSolder, F.Cu at (133.3, 96.0)
- added J2: USB_A, Connector_USB:USB_A_Molex_67643_Horizontal, F.Cu at (146.8, 90.8)
- added J3: Conn_01x03, Connector_PinSocket_2.54mm:PinSocket_1x03_P2.54mm_Vertical, F.Cu at (147.5, 82.2)
- added R2: 130, Resistor_SMD:R_1206_3216Metric_Pad1.30x1.75mm_HandSolder, F.Cu at (130.2, 89.4)
- added R3: 130, Resistor_SMD:R_1206_3216Metric_Pad1.30x1.75mm_HandSolder, F.Cu at (126.8, 89.4)
- added R4: 130, Resistor_SMD:R_1206_3216Metric_Pad1.30x1.75mm_HandSolder, F.Cu at (123.4, 89.4)
- added R5: 130, Resistor_SMD:R_1206_3216Metric_Pad1.30x1.75mm_HandSolder, F.Cu at (133.4, 89.4)
- added SW1: SW_DPDT_x2, MMS_footprints:SW_MTS102_3Pins_2Positions, F.Cu at (127.9, 56.8)
- added SW2: SW_DPDT_x2, MMS_footprints:SW_MTS102_3Pins_2Positions, F.Cu at (127.9, 68.0)
- added SW3: SW_DPDT_x2, MMS_footprints:SW_MTS102_3Pins_2Positions, F.Cu at (127.9, 79.2)
- added SW4: SW_DIP_x01, Button_Switch_THT:SW_PUSH_6mm, F.Cu at (157.9, 65.0)
- added SW6: SW_DIP_x01, Button_Switch_THT:SW_PUSH_6mm, F.Cu at (147.3, 65.0)
- added U1: NRF24L01_Breakout, RF_Module:nRF24L01_Breakout, F.Cu at (114.0, 56.4)
Routing:
- net /GPIO16: track 0.00 -> 65.7 mm
- net /GPIO23: track 0.00 -> 65.4 mm
- net /GPIO26: track 0.00 -> 61.9 mm
- net /GPIO25: track 0.00 -> 61.6 mm
- net +3.3VA: track 0.00 -> 50.7 mm
- net /GPIO8/SPI0.CE0: track 0.00 -> 42.5 mm, vias 0 -> 1
- net /GPIO10/SPI0.MOSI: track 0.00 -> 41.1 mm, vias 0 -> 1
- net /GPIO24: track 0.00 -> 37.7 mm
- net /GPIO5: track 0.00 -> 35.1 mm
- net /GPIO9/SPI0.MISO: track 0.00 -> 32.2 mm
- net /GPIO11/SPI0.SCLK: track 0.00 -> 32.0 mm
- net /GPIO27: track 0.00 -> 21.0 mm, vias 0 -> 2
- net /GPIO6: track 0.00 -> 18.6 mm
- net /GPIO19/PCM.FS: track 0.00 -> 18.5 mm
- net /GPIO22: track 0.00 -> 17.8 mm
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- added copper zone on B.Cu, net GND
- added copper zone on F.Cu, net GND
Other:
- outline, holes or cut-outs redrawn
- board text removed: "CAMERA (OPTIONAL)"
