File: MTP_PCB/_autosave-MTP_PCB.kicad_sch (KiCad schematic)
At the start: 17 parts, among them J1 GPIO, J2 USB_A, J3 Conn_01x03, SW1 SW_DPDT_x2, SW2 SW_DPDT_x2, SW3 SW_DPDT_x2, SW4 SW_DIP_x01, SW6 SW_DIP_x01, U1 NRF24L01_Breakout

Commit message: first version PCB finished
Connections:
- net +5V: no longer J2.1 (VBUS), J3.1 (Pin_1)
- new net +5VA: J2.1 (VBUS), J3.1 (Pin_1)
Changed lines of the file:
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@@
   (junction (at 76.2 43.18) (diameter 1.016) (color 0 0 0 0)
   )
+  (junction (at 76.2 25.4) (diameter 0) (color 0 0 0 0)
+  )
   (junction (at 232.41 34.29) (diameter 0) (color 0 0 0 0)
   )
@@
   (junction (at 143.51 62.23) (diameter 0) (color 0 0 0 0)
   )
-  (junction (at 166.37 44.45) (diameter 0) (color 0 0 0 0)
+  (junction (at 165.1 44.45) (diameter 0) (color 0 0 0 0)
   )
   (junction (at 76.2 63.5) (diameter 1.016) (color 0 0 0 0)
@@
     (stroke (width 0) (type solid))
   )
-  (wire (pts (xy 166.37 44.45) (xy 177.8 44.45))
-    (stroke (width 0) (type default))
-  )
   (wire (pts (xy 76.2 50.8) (xy 76.2 63.5))
     (stroke (width 0) (type solid))
@@
     (stroke (width 0) (type solid))
   )
-  (wire (pts (xy 156.21 44.45) (xy 166.37 44.45))
+  (wire (pts (xy 156.21 44.45) (xy 165.1 44.45))
     (stroke (width 0) (type default))
   )
@@
     (stroke (width 0) (type default))
   )
-  (wire (pts (xy 76.2 24.13) (xy 76.2 27.94))
-    (stroke (width 0) (type solid))
+  (wire (pts (xy 76.2 24.13) (xy 76.2 25.4))
+    (stroke (width 0) (type solid))
+  )
+  (wire (pts (xy 165.1 44.45) (xy 177.8 44.45))
+    (stroke (width 0) (type default))
   )
   (wire (pts (xy 31.75 35.56) (xy 60.96 35.56))
@@
   )
   (wire (pts (xy 73.66 71.12) (xy 100.33 71.12))
+    (stroke (width 0) (type solid))
+  )
+  (wire (pts (xy 76.2 25.4) (xy 76.2 27.94))
     (stroke (width 0) (type solid))
   )
@@
     )
   )
-  (symbol (lib_id "power:+5V") (at 166.37 44.45 0) (unit 1)
-    (in_bom yes) (on_board yes) (dnp no)
-    (property "Reference" "#PWR019" (at 166.37 48.26 0)
-      (effects (font (size 1.27 1.27)) hide)
-    )
-    (property "Value" "+5V" (at 166.7383 40.1256 0)
-      (effects (font (size 1.27 1.27)))
-    )
-    (property "Footprint" "" (at 166.37 44.45 0)
-      (effects (font (size 1.27 1.27)))
-    )
-    (property "Datasheet" "" (at 166.37 44.45 0)
-      (effects (font (size 1.27 1.27)))
-    )
-    (pin "1")
-    (instances
-      (project "MTP_PCB"
-        (path "/e63e39d7-6ac0-4ffd-8aa3-1841a4541b55"
-          (reference "#PWR019") (unit 1)
-        )
-      )
-    )
-  )
   (symbol (lib_name "GND_1") (lib_id "power:GND") (at 68.58 142.24 0) (unit 1)
     (in_bom yes) (on_board yes) (dnp no) (fields_autoplaced)
@@
     )
   )
+  (symbol (lib_id "power:PWR_FLAG") (at 76.2 25.4 270) (unit 1)
+    (in_bom yes) (on_board yes) (dnp no) (fields_autoplaced)
+    (property "Reference" "#FLG02" (at 78.105 25.4 0)
+      (effects (font (size 1.27 1.27)) hide)
+    )
+    (property "Value" "PWR_FLAG" (at 80.01 26.035 90)
+      (effects (font (size 1.27 1.27)) (justify left))
+    )
+    (property "Footprint" "" (at 76.2 25.4 0)
+      (effects (font (size 1.27 1.27)) hide)
+    )
+    (property "Datasheet" "~" (at 76.2 25.4 0)
+      (effects (font (size 1.27 1.27)) hide)
+    )
+    (pin "1")
+    (instances
+      (project "MTP_PCB"
+        (path "/e63e39d7-6ac0-4ffd-8aa3-1841a4541b55"
+          (reference "#FLG02") (unit 1)
+        )
+      )
+    )
+  )
   (symbol (lib_id "Switch:SW_DPDT_x2") (at 45.72 133.35 90) (unit 1)
     (in_bom yes) (on_board yes) (dnp no) (fields_autoplaced)
@@
         )
       )
+    )
+  )
+  (symbol (lib_id "power:+5VA") (at 165.1 44.45 0) (unit 1)
+    (in_bom yes) (on_board yes) (dnp no) (fields_autoplaced)
+    (property "Reference" "#PWR019" (at 165.1 48.26 0)
+      (effects (font (size 1.27 1.27)) hide)
+    )
+    (property "Value" "+5VA" (at 165.1 40.64 0)
+      (effects (font (size 1.27 1.27)))
+    )
+    (property "Footprint" "" (at 165.1 44.45 0)
+      (effects (font (size 1.27 1.27)) hide)
+    )
+    (property "Datasheet" "" (at 165.1 44.45 0)
+      (effects (font (size 1.27 1.27)) hide)
+    )
+    (pin "1")
+    (instances
+      (project "MTP_PCB"
+        (path "/e63e39d7-6ac0-4ffd-8aa3-1841a4541b55"
+          (reference "#PWR019") (unit 1)
+        )
+      )
